File: schematics/full-schematic/Memory.sch (KiCad schematic (older format))
At the start: 0 parts

Commit message: Schematics
Parts:
- added C10, C11: 0.1u, Capacitor_SMD:C_0603_1608Metric_Pad1.05x0.95mm_HandSolder, symbol Device:C
- added R10, R11, R12, R13, R14, R2, R9: 1k, Resistor_SMD:R_0603_1608Metric_Pad1.05x0.95mm_HandSolder, symbol Device:R
- added U13: CY62128ELL-45SXI, Package_DIP:DIP-32_W15.24mm_SMDSocket_SmallPads, symbol z80-project:CY62128ELL-45SXI
- added U14: AT28C64B-15PU, Package_DIP:DIP-28_W15.24mm_Socket, symbol z80-project:AT28C64B-15PU
Connections:
- new net: R9.1, U13.10 (A16)
- new net: R2.1, U13.6 (CE2)
- new net: R14.1, U14.2 (A12)
- new net: R12.1, U14.21 (A10)
- new net: R13.1, U14.23 (A11)
- new net: R11.1, U14.24 (A9)
- new net: R10.1, U14.25 (A8)
- new net +5V: C10.1, C11.1, R2.2, U13.8 (VCC), U14.28 (VCC)
- new net -MRD-: U13.32 (-OE-), U14.22 (-OE-)
- new net -MWR-: U13.5 (-WE-), U14.27 (-WE-)
- new net -ROMCS-: U14.20 (-CE-)
- new net A0: U13.20 (A0), U14.10 (A0)
- new net A1: U13.19 (A1), U14.9 (A1)
- new net A10: U13.31 (A10)
- new net A11: U13.1 (A11)
- new net A12: U13.12 (A12)
- new net A13: U13.4 (A13)
- new net A14: U13.11 (A14)
- new net A15: U13.7 (A15)
- new net A2: U13.18 (A2), U14.8 (A2)
- new net A3: U13.17 (A3), U14.7 (A3)
- new net A4: U13.16 (A4), U14.6 (A4)
- new net A5: U13.15 (A5), U14.5 (A5)
- new net A6: U13.14 (A6), U14.4 (A6)
- new net A7: U13.13 (A7), U14.3 (A7)
- new net A8: U13.3 (A8)
- new net A9: U13.2 (A9)
- new net D0: U13.21 (D0), U14.11 (D0)
- new net D1: U13.22 (D1), U14.12 (D1)
- new net D2: U13.23 (D2), U14.13 (D2)
- new net D3: U13.25 (D3), U14.15 (D3)
- new net D4: U13.26 (D4), U14.16 (D4)
- new net D5: U13.27 (D5), U14.17 (D5)
- new net D6: U13.28 (D6), U14.18 (D6)
- new net D7: U13.29 (D7), U14.19 (D7)
- new net GND: C10.2, C11.2, R10.2, R11.2, R12.2, R13.2, R14.2, R9.2, U13.24 (GND), U14.14 (GND)
