File: schematics/full-schematic/Memory.sch (KiCad schematic (older format))
At the start: 11 parts, among them U13 CY62128ELL-45SXI, U14 AT28C64B-15PU

Commit message: Schematic updates
Parts:
- removed R10, R12, R13, R14: 1k, Resistor_SMD:R_0603_1608Metric_Pad1.05x0.95mm_HandSolder, symbol Device:R
- removed U14: AT28C64B-15PU, Package_DIP:DIP-28_W15.24mm_Socket, symbol z80-project:AT28C64B-15PU
- added JP1: Jumper_NC_Dual, Connector_PinHeader_2.54mm:PinHeader_1x03_P2.54mm_Vertical_SMD_Pin1Left, symbol Device:Jumper_NC_Dual
- added U14: AT28C256-15PU, Package_DIP:DIP-28_W15.24mm_Socket_LongPads, symbol z80-project:AT28C256-15PU
- renumbered R9 to R10, R2 to R9
Connections:
- net +5V: now also R11.1, U14.28 (VCC)
- net -ROMCS-: now also U14.20 (-CE-)
- net A0: now also U14.10 (A0)
- net A1: now also U14.9 (A1)
- net A10: now also U14.21 (A10)
- net A11: now also U14.23 (A11)
- net A12: now also U14.2 (A12)
- net A13: now also U14.26 (A13)
- net A14: now also U14.1 (A14)
- net A2: now also U14.8 (A2)
- net A3: now also U14.7 (A3)
- net A4: now also U14.6 (A4)
- net A5: now also U14.5 (A5)
- net A6: now also U14.4 (A6)
- net A7: now also U14.3 (A7)
- net A8: now also U14.25 (A8)
- net A9: now also U14.24 (A9)
- net D0: now also U14.11 (D0)
- net D1: now also U14.12 (D1)
- net D2: now also U14.13 (D2)
- net D3: now also U14.15 (D3)
- net D4: now also U14.16 (D4)
- net D5: now also U14.17 (D5)
- net D6: now also U14.18 (D6)
- net D7: now also U14.19 (D7)
- net GND: now also U14.14 (GND); no longer R11.2
- net -RAMCS-: now reaches U13.30 (-CE1-)
- net -MRD- renamed -RD-
- net -RD-: now also U14.22 (-OE-)
- net -MWR- renamed -WR-
- net -WR-: now also JP1.1
- new net: JP1.2, U14.27 (-WE-)
- new net: JP1.3, R11.2
Other:
- moved on the sheet: C11
