File: schematics/full-schematic/full-schematic.kicad_pcb (KiCad board)
At the start: 2 copper layers, 34 parts, among them SW2 SW_Push_Dual, SW3 SW_Push_Dual, U1 L7805, U10 74LS04, U11 74LS109, U12 74LS08, U2 74LS04, U3 Z80CPU, U4 74LS32, U5 LP3470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

Commit message: Schematics
Parts:
- added C10: 0.1u, Capacitor_SMD:C_0603_1608Metric_Pad1.05x0.95mm_HandSolder, F.Cu at (315.0, 169.7)
- added C11: 0.1u, Capacitor_SMD:C_0603_1608Metric_Pad1.05x0.95mm_HandSolder, F.Cu at (319.3, 169.7)
- added R10: 1k, Resistor_SMD:R_0603_1608Metric_Pad1.05x0.95mm_HandSolder, F.Cu at (332.4, 169.7)
- added R11: 1k, Resistor_SMD:R_0603_1608Metric_Pad1.05x0.95mm_HandSolder, F.Cu at (336.7, 169.7)
- added R12: 1k, Resistor_SMD:R_0603_1608Metric_Pad1.05x0.95mm_HandSolder, F.Cu at (315.0, 172.2)
- added R13: 1k, Resistor_SMD:R_0603_1608Metric_Pad1.05x0.95mm_HandSolder, F.Cu at (319.3, 172.2)
- added R14: 1k, Resistor_SMD:R_0603_1608Metric_Pad1.05x0.95mm_HandSolder, F.Cu at (323.7, 172.2)
- added R2: 1k, Resistor_SMD:R_0603_1608Metric_Pad1.05x0.95mm_HandSolder, F.Cu at (323.7, 169.7)
- added R9: 1k, Resistor_SMD:R_0603_1608Metric_Pad1.05x0.95mm_HandSolder, F.Cu at (328.0, 169.7)
- added TP1: TestPoint_Probe, TestPoint:TestPoint_Pad_D1.5mm, F.Cu at (376.9, 177.3)
- added TP2: TestPoint_Probe, TestPoint:TestPoint_Pad_D1.5mm, F.Cu at (376.9, 170.2)
- added TP3: TestPoint_Probe, TestPoint:TestPoint_Pad_D1.5mm, F.Cu at (380.5, 170.2)
- added U13: CY62128ELL-45SXI, Package_DIP:DIP-32_W15.24mm_SMDSocket_SmallPads, F.Cu at (303.1, 189.6)
- added U14: AT28C64B-15PU, Package_DIP:DIP-28_W15.24mm_Socket, F.Cu at (348.0, 179.8)
- moved U5 18.6 mm to (333.2, 158.0)
Connections:
- net /RST renamed RST
- D1 pad 1: Net-(D1-Pad1) -> (no net)
- D1 pad 2: +VDC -> (no net)
- U11 pad 7: Net-(U11-Pad7) -> (no net)
- U2 pad 4: /-RST- -> -RST-
- U2 pad 6: /SW_CLK -> (no net)
- U3 pad 16: Net-(U3-Pad16) -> (no net)
- U3 pad 17: Net-(U3-Pad17) -> (no net)
- U3 pad 18: Net-(U3-Pad18) -> (no net)
- U3 pad 23: Net-(U3-Pad23) -> (no net)
- U3 pad 24: Net-(U3-Pad24) -> (no net)
- U3 pad 25: Net-(U3-Pad25) -> (no net)
- U3 pad 28: Net-(U3-Pad28) -> (no net)
- U5 pad 5: (no net) -> Net-(D3-Pad1)
- U6 pad 6: -RAMCS- -> (no net)
- U8 pad 10: -IOCS5- -> (no net)
- U8 pad 11: -IOCS4- -> (no net)
- U8 pad 12: -IOCS3- -> (no net)
- U8 pad 13: -IOCS2- -> (no net)
- U8 pad 14: -IOCS1- -> (no net)
- U8 pad 15: -IOCS0- -> (no net)
- U8 pad 9: -IOCS6- -> (no net)
- X1 pad 5: /OSC_CLK -> (no net)
