File: schematics/full-schematic/full-schematic.kicad_pcb (KiCad board)
At the start: 2 copper layers, 48 parts, among them SW2 SW_Push_Dual, SW3 SW_Push_Dual, U1 L7805, U10 74LS04, U11 74LS109, U12 74LS08, U13 CY62128ELL-45SXI, U14 AT28C64B-15PU, U2 74LS04, U3 Z80CPU, U4 74LS32, U5 LP3470, U6 74LS32, U7 74LS32, U8 74LS138, U9 74LS32, X1 CXO_DIP8

Commit message: Schematic updates
Parts:
- removed C1, C10, C11, C4, C5, C6, C7, C8, C9: 0.1u, Capacitor_SMD:C_0603_1608Metric_Pad1.05x0.95mm_HandSolder
- removed C2, C3: 1m, Capacitor_SMD:C_0603_1608Metric_Pad1.05x0.95mm_HandSolder
- removed D1, D3: D_Schottky, Diode_SMD:D_0603_1608Metric_Pad1.05x0.95mm_HandSolder
- removed D2: LED, LED_SMD:LED_0603_1608Metric_Pad1.05x0.95mm_HandSolder
- removed R1: 330, Resistor_SMD:R_0603_1608Metric_Pad1.05x0.95mm_HandSolder
- removed R10, R11, R12, R13, R14, R2, R4, R8, R9: 1k, Resistor_SMD:R_0603_1608Metric_Pad1.05x0.95mm_HandSolder
- removed R3, R7: 10k, Resistor_SMD:R_0603_1608Metric_Pad1.05x0.95mm_HandSolder
- removed R5, R6: 100k, Resistor_SMD:R_0603_1608Metric_Pad1.05x0.95mm_HandSolder
- removed SW2, SW3: SW_Push_Dual, Button_Switch_SMD:SW_MEC_5GSH9
- removed TP1, TP2, TP3: TestPoint_Probe, TestPoint:TestPoint_Pad_D1.5mm
- removed U1: L7805, Package_TO_SOT_SMD:TO-263-2
- removed U10, U2: 74LS04, Package_SO:SOIC-14_3.9x8.7mm_P1.27mm
- removed U11: 74LS109, Package_DIP:DIP-16_W7.62mm
- removed U12: 74LS08, Package_SO:SOIC-14_3.9x8.7mm_P1.27mm
- removed U13: CY62128ELL-45SXI, Package_DIP:DIP-32_W15.24mm_SMDSocket_SmallPads
- removed U14: AT28C64B-15PU, Package_DIP:DIP-28_W15.24mm_Socket
- removed U3: Z80CPU, Package_DIP:DIP-40_W15.24mm
- removed U4, U6, U7, U9: 74LS32, Package_SO:SOIC-14_3.9x8.7mm_P1.27mm
- removed U5: LP3470, Package_TO_SOT_SMD:SOT-23-5_HandSoldering
- removed U8: 74LS138, Package_SO:SOIC-16_3.9x9.9mm_P1.27mm
- removed X1: CXO_DIP8, Oscillator:Oscillator_DIP-8

Commit message: Stuff
Parts:
- added C1: 0.1u, Capacitor_SMD:C_0603_1608Metric_Pad1.05x0.95mm_HandSolder, F.Cu at (230.4, 55.8)
- added C10: 0.1u, Capacitor_SMD:C_0603_1608Metric_Pad1.05x0.95mm_HandSolder, F.Cu at (395.9, 95.6)
- added C11: 0.1u, Capacitor_SMD:C_0603_1608Metric_Pad1.05x0.95mm_HandSolder, F.Cu at (343.8, 144.4)
- added C12: 0.1u, Capacitor_SMD:C_0603_1608Metric_Pad1.05x0.95mm_HandSolder, F.Cu at (322.1, 146.9)
- added C2: 0.1u, Capacitor_SMD:C_0603_1608Metric_Pad1.05x0.95mm_HandSolder, F.Cu at (199.9, 70.4)
- added C3: 0.1u, Capacitor_SMD:C_0603_1608Metric_Pad1.05x0.95mm_HandSolder, F.Cu at (320.7, 73.7)
- added C4: 0.1u, Capacitor_SMD:C_0603_1608Metric_Pad1.05x0.95mm_HandSolder, F.Cu at (320.7, 76.2)
- added C5: 1m, Capacitor_SMD:C_0603_1608Metric_Pad1.05x0.95mm_HandSolder, F.Cu at (325.0, 76.1)
- added C6: 1m, Capacitor_SMD:C_0603_1608Metric_Pad1.05x0.95mm_HandSolder, F.Cu at (316.3, 78.7)
- added C7: 0.1u, Capacitor_SMD:C_0603_1608Metric_Pad1.05x0.95mm_HandSolder, F.Cu at (320.7, 78.7)
- added C8: 0.1u, Capacitor_SMD:C_0603_1608Metric_Pad1.05x0.95mm_HandSolder, F.Cu at (316.3, 81.2)
- added C9: 0.1u, Capacitor_SMD:C_0603_1608Metric_Pad1.05x0.95mm_HandSolder, F.Cu at (448.9, 67.6)
- added D1: D_Schottky, Diode_SMD:D_0603_1608Metric_Pad1.05x0.95mm_HandSolder, F.Cu at (320.8, 71.2)
- added D2: LED, LED_SMD:LED_0603_1608Metric_Pad1.05x0.95mm_HandSolder, F.Cu at (316.4, 71.2)
- added D3: LED, LED_SMD:LED_0603_1608Metric_Pad1.05x0.95mm_HandSolder, F.Cu at (317.7, 144.4)
- added J1: Conn_02x25_Top_Bottom, z80-project:Molex_553595029_CF_Socket, F.Cu at (322.0, 137.7)
- added J2: Conn_01x02, Connector_PinHeader_2.54mm:PinHeader_1x02_P2.54mm_Vertical, F.Cu at (307.4, 145.4)
- added J3: Conn_01x04, Connector_PinHeader_2.54mm:PinHeader_1x04_P2.54mm_Vertical, F.Cu at (298.1, 145.4)
- added J4: Conn_01x02, Connector_PinHeader_2.54mm:PinHeader_1x02_P2.54mm_Vertical, F.Cu at (302.7, 147.9)
- added JP1: Jumper_NC_Dual, Connector_PinHeader_2.54mm:PinHeader_1x03_P2.54mm_Vertical_SMD_Pin1Left, F.Cu at (453.3, 56.9)
- added R1: 100k, Resistor_SMD:R_0603_1608Metric_Pad1.05x0.95mm_HandSolder, F.Cu at (325.1, 73.6)
- added R10: 1k, Resistor_SMD:R_0603_1608Metric_Pad1.05x0.95mm_HandSolder, F.Cu at (459.5, 53.2)
- added R11: 1k, Resistor_SMD:R_0603_1608Metric_Pad1.05x0.95mm_HandSolder, F.Cu at (413.3, 95.6)
- added R12: 1k, Resistor_SMD:R_0603_1608Metric_Pad1.05x0.95mm_HandSolder, F.Cu at (408.9, 95.6)
- added R13: 1k, Resistor_SMD:R_0603_1608Metric_Pad1.05x0.95mm_HandSolder, F.Cu at (404.6, 95.6)
- added R14: 1k, Resistor_SMD:R_0603_1608Metric_Pad1.05x0.95mm_HandSolder, F.Cu at (400.2, 95.6)
- added R15: 1k, Resistor_SMD:R_0603_1608Metric_Pad1.05x0.95mm_HandSolder, F.Cu at (322.1, 144.4)
- added R16: 1k, Resistor_SMD:R_0603_1608Metric_Pad1.05x0.95mm_HandSolder, F.Cu at (326.4, 144.4)
- added R17: 1k, Resistor_SMD:R_0603_1608Metric_Pad1.05x0.95mm_HandSolder, F.Cu at (330.8, 144.4)
- added R18: 1k, Resistor_SMD:R_0603_1608Metric_Pad1.05x0.95mm_HandSolder, F.Cu at (335.1, 144.4)
- added R19: 1k, Resistor_SMD:R_0603_1608Metric_Pad1.05x0.95mm_HandSolder, F.Cu at (339.5, 144.4)
- added R2: 10k, Resistor_SMD:R_0603_1608Metric_Pad1.05x0.95mm_HandSolder, F.Cu at (234.1, 53.1)
- added R3: 10k, Resistor_SMD:R_0603_1608Metric_Pad1.05x0.95mm_HandSolder, F.Cu at (316.3, 83.8)
- added R4: 330, Resistor_SMD:R_0603_1608Metric_Pad1.05x0.95mm_HandSolder, F.Cu at (316.3, 86.3)
- added R5: 1k, Resistor_SMD:R_0603_1608Metric_Pad1.05x0.95mm_HandSolder, F.Cu at (343.6, 69.9)
- added R6: 1k, Resistor_SMD:R_0603_1608Metric_Pad1.05x0.95mm_HandSolder, F.Cu at (320.7, 83.8)
- added R7: 1k, Resistor_SMD:R_0603_1608Metric_Pad1.05x0.95mm_HandSolder, F.Cu at (316.3, 88.8)
- added R8: 1k, Resistor_SMD:R_0603_1608Metric_Pad1.05x0.95mm_HandSolder, F.Cu at (325.0, 78.7)
- added R9: 1k, Resistor_SMD:R_0603_1608Metric_Pad1.05x0.95mm_HandSolder, F.Cu at (421.0, 90.5)
- added SW1: SW_Push_Dual, Button_Switch_THT:SW_PUSH_6mm, F.Cu at (343.7, 80.5)
- added SW2: SW_SPST, Button_Switch_THT:SW_E-Switch_EG1224_SPDT_Angled, F.Cu at (318.0, 55.6)
- added TP1: TestPoint_Probe, TestPoint:TestPoint_Pad_D1.5mm, F.Cu at (203.7, 67.1)
- added TP2: TestPoint_Probe, TestPoint:TestPoint_Pad_D1.5mm, F.Cu at (329.0, 76.7)
- added TP3: TestPoint_Probe, TestPoint:TestPoint_Pad_D1.5mm, F.Cu at (463.4, 53.8)
- added U1: LP3470, Package_TO_SOT_SMD:SOT-23-5_HandSoldering, F.Cu at (233.7, 55.9)
- added U10: 74HC107D, Package_SO:SOIC-14_3.9x8.7mm_P1.27mm, F.Cu at (445.1, 57.1)
- added U11: 74LVC1G32, Package_TO_SOT_SMD:SOT-23-5_HandSoldering, F.Cu at (435.3, 75.1)
- added U12: 74LVC1G04, Package_TO_SOT_SMD:SOT-23-5_HandSoldering, F.Cu at (435.3, 70.4)
- added U13: 74LVC1G32, Package_TO_SOT_SMD:SOT-23-5_HandSoldering, F.Cu at (452.2, 64.1)
- added U14: 74LVC1G32, Package_TO_SOT_SMD:SOT-23-5_HandSoldering, F.Cu at (441.1, 69.2)
- added U15: AT28C256-15PU, Package_DIP:DIP-28_W15.24mm_Socket_LongPads, F.Cu at (415.1, 54.1)
- added U16: PCF8584, Package_SO:SOIC-20W_7.5x12.8mm_P1.27mm, F.Cu at (371.4, 115.6)
- added U17: CP82C52Z, Package_DIP:DIP-28_W15.24mm, F.Cu at (348.2, 110.5)
- added U18: 74LVC1G04, Package_TO_SOT_SMD:SOT-23-5_HandSoldering, F.Cu at (312.6, 145.4)
- added U2: 74LVC1G08, Package_TO_SOT_SMD:SOT-23-5_HandSoldering, F.Cu at (332.7, 66.7)
- added U3: L7805, Package_TO_SOT_SMD:TO-263-2, F.Cu at (338.6, 58.2)
- added U4: Z80CPU, Package_DIP:DIP-40_W15.24mm, F.Cu at (297.3, 54.1)
- added U5: 74LS138, Package_SO:SOIC-16_3.9x9.9mm_P1.27mm, F.Cu at (436.7, 57.7)
- added U6: CY62128ELL-45SXI, Package_DIP:DIP-32_W15.24mm_SMDSocket_SmallPads, F.Cu at (403.4, 73.2)
- added U7: 74LVC1G32, Package_TO_SOT_SMD:SOT-23-5_HandSoldering, F.Cu at (443.8, 64.5)
- added U8: 74LVC1G32, Package_TO_SOT_SMD:SOT-23-5_HandSoldering, F.Cu at (435.3, 65.8)
- added U9: 74LVC1G08, Package_TO_SOT_SMD:SOT-23-5_HandSoldering, F.Cu at (415.9, 91.6)
- added X1: XO32, Oscillator:Oscillator_SMD_EuroQuartz_XO32-4Pin_3.2x2.5mm, F.Cu at (199.9, 67.8)
