File: schematics/full-schematic/CPU.sch (KiCad schematic (older format))
At the start: 13 parts, among them U10 74LS04, U11 74LS109, U12 74LS08, U2 74LS04, U3 Z80CPU, U4 74LS32, U6 74LS32, U7 74LS32, U8 74LS138, U9 74LS32

Commit message: Schematics
Parts:
- added TP1: TestPoint_Probe, TestPoint:TestPoint_Pad_D1.5mm, symbol Connector:TestPoint_Probe
- R4, R8: footprint (none) -> Resistor_SMD:R_0603_1608Metric_Pad1.05x0.95mm_HandSolder
- U11: footprint (none) -> Package_DIP:DIP-16_W7.62mm
- U12, U4, U6, U7, U9: footprint (none) -> Package_SO:SOIC-14_3.9x8.7mm_P1.27mm
- U3: footprint (none) -> Package_DIP:DIP-40_W15.24mm
- U8: footprint (none) -> Package_SO:SOIC-16_3.9x9.9mm_P1.27mm
Connections:
- net ROMDis: now also TP1.1
Changed lines of the file:
@@
 EESchema Schematic File Version 4
-LIBS:full-schematic-cache
-EELAYER 29 0
+EELAYER 30 0
 EELAYER END
 $Descr A4 11693 8268
 encoding utf-8
-Sheet 2 3
+Sheet 2 4
 Title ""
 Date ""
@@
 Comment4 ""
 $EndDescr
-$Comp
-L CPU:Z80CPU U?
-U 1 1 5D5CF86D
-P 3200 5350
-AR Path="/5D5CF86D" Ref="U?"  Part="1"
-AR Path="/5D5CBDC9/5D5CF86D" Ref="U3"  Part="1"
-F 0 "U3" H 2900 6750 50  0000 C CNN
-F 1 "Z80CPU" H 3450 6750 50  0000 C CNN
-F 2 "" H 3200 5750 50  0001 C CNN
-F 3 "www.zilog.com/manage_directlink.php?filepath=docs/z80/um0080" H 3200 5750 50  0001 C CNN
-	1    3200 5350
-	1    0    0    -1
-$EndComp
 Wire Wire Line
 	2500 4150 2150 4150
@@
 F 0 "U4" H 9200 5000 50  0000 C CNN
 F 1 "74LS32" H 9500 5000 50  0000 C CNN
-F 2 "" H 9300 4800 50  0001 C CNN
+F 2 "Package_SO:SOIC-14_3.9x8.7mm_P1.27mm" H 9300 4800 50  0001 C CNN
 F 3 "http://www.ti.com/lit/gpn/sn74LS32" H 9300 4800 50  0001 C CNN
 	3    9300 4800
@@
 F 0 "U4" H 9200 5000 50  0000 C CNN
 F 1 "74LS32" H 9500 5000 50  0000 C CNN
-F 2 "" H 9300 5200 50  0001 C CNN
+F 2 "Package_SO:SOIC-14_3.9x8.7mm_P1.27mm" H 9300 5200 50  0001 C CNN
 F 3 "http://www.ti.com/lit/gpn/sn74LS32" H 9300 5200 50  0001 C CNN
 	4    9300 5200
@@
 F 0 "U6" H 1850 1900 50  0000 C CNN
 F 1 "74LS32" H 2150 1900 50  0000 C CNN
-F 2 "" H 1950 1700 50  0001 C CNN
+F 2 "Package_SO:SOIC-14_3.9x8.7mm_P1.27mm" H 1950 1700 50  0001 C CNN
 F 3 "http://www.ti.com/lit/gpn/sn74LS32" H 1950 1700 50  0001 C CNN
 	3    1950 1700
@@
 F 0 "U8" H 3150 1950 50  0000 C CNN
 F 1 "74LS138" H 3550 1950 50  0000 C CNN
-F 2 "" H 3350 1500 50  0001 C CNN
+F 2 "Package_SO:SOIC-16_3.9x9.9mm_P1.27mm" H 3350 1500 50  0001 C CNN
 F 3 "http://www.ti.com/lit/gpn/sn74LS138" H 3350 1500 50  0001 C CNN
 	1    3350 1500
@@
 F 0 "U11" H 6300 2250 50  0000 C CNN
 F 1 "74LS109" H 6700 2250 50  0000 C CNN
-F 2 "" H 6500 2000 50  0001 C CNN
+F 2 "Package_DIP:DIP-16_W7.62mm" H 6500 2000 50  0001 C CNN
 F 3 "http://www.ti.com/lit/gpn/sn74LS109" H 6500 2000 50  0001 C CNN
 	1    6500 2000
@@
 F 0 "R8" H 6570 1496 50  0000 L CNN
 F 1 "1k" H 6570 1405 50  0000 L CNN
-F 2 "" V 6430 1450 50  0001 C CNN
+F 2 "Resistor_SMD:R_0603_1608Metric_Pad1.05x0.95mm_HandSolder" V 6430 1450 50  0001 C CNN
 F 3 "~" H 6500 1450 50  0001 C CNN
 	1    6500 1450
@@
 	1    0    0    -1
 $EndComp
-Wire Wire Line
-	6800 1900 7350 1900
 Text Label 7200 1900 2    50   ~ 0
 ROMDis
@@
 F 0 "U4" H 9200 4050 50  0000 C CNN
 F 1 "74LS32" H 9500 4050 50  0000 C CNN
-F 2 "" H 9300 4250 50  0001 C CNN
+F 2 "Package_SO:SOIC-14_3.9x8.7mm_P1.27mm" H 9300 4250 50  0001 C CNN
 F 3 "http://www.ti.com/lit/gpn/sn74LS32" H 9300 4250 50  0001 C CNN
 	2    9300 4250
@@
 F 0 "U4" H 9200 4050 50  0000 C CNN
 F 1 "74LS32" H 9500 4050 50  0000 C CNN
-F 2 "" H 9300 3850 50  0001 C CNN
+F 2 "Package_SO:SOIC-14_3.9x8.7mm_P1.27mm" H 9300 3850 50  0001 C CNN
 F 3 "http://www.ti.com/lit/gpn/sn74LS32" H 9300 3850 50  0001 C CNN
 	1    9300 3850
@@
 F 0 "R4" V 6150 2050 50  0000 C CNN
 F 1 "1k" V 6150 2200 50  0000 C CNN
-F 2 "" V 5980 2100 50  0001 C CNN
+F 2 "Resistor_SMD:R_0603_1608Metric_Pad1.05x0.95mm_HandSolder" V 5980 2100 50  0001 C CNN
 F 3 "~" H 6050 2100 50  0001 C CNN
 	1    6050 2100
@@
 F 0 "U9" H 4850 2200 50  0000 C CNN
 F 1 "74LS32" H 5150 2200 50  0000 C CNN
-F 2 "" H 4950 2000 50  0001 C CNN
+F 2 "Package_SO:SOIC-14_3.9x8.7mm_P1.27mm" H 4950 2000 50  0001 C CNN
 F 3 "http://www.ti.com/lit/gpn/sn74LS32" H 4950 2000 50  0001 C CNN
 	3    4950 2000
@@
 F 0 "U7" H 4850 2750 50  0000 C CNN
 F 1 "74LS32" H 5150 2750 50  0000 C CNN
-F 2 "" H 4950 2550 50  0001 C CNN
+F 2 "Package_SO:SOIC-14_3.9x8.7mm_P1.27mm" H 4950 2550 50  0001 C CNN
 F 3 "http://www.ti.com/lit/gpn/sn74LS32" H 4950 2550 50  0001 C CNN
 	3    4950 2550
@@
 F 0 "U12" H 5450 2850 50  0000 C CNN
 F 1 "74LS08" H 5750 2850 50  0000 C CNN
-F 2 "" H 5550 2650 50  0001 C CNN
+F 2 "Package_SO:SOIC-14_3.9x8.7mm_P1.27mm" H 5550 2650 50  0001 C CNN
 F 3 "http://www.ti.com/lit/gpn/sn74LS08" H 5550 2650 50  0001 C CNN
 	1    5550 2650
@@
 F 0 "U9" H 7550 2200 50  0000 C CNN
 F 1 "74LS32" H 7850 2200 50  0000 C CNN
-F 2 "" H 7650 2000 50  0001 C CNN
+F 2 "Package_SO:SOIC-14_3.9x8.7mm_P1.27mm" H 7650 2000 50  0001 C CNN
 F 3 "http://www.ti.com/lit/gpn/sn74LS32" H 7650 2000 50  0001 C CNN
 	1    7650 2000
@@
 F 0 "U6" H 9150 2300 50  0000 C CNN
 F 1 "74LS32" H 9450 2300 50  0000 C CNN
-F 2 "" H 9250 2500 50  0001 C CNN
+F 2 "Package_SO:SOIC-14_3.9x8.7mm_P1.27mm" H 9250 2500 50  0001 C CNN
 F 3 "http://www.ti.com/lit/gpn/sn74LS32" H 9250 2500 50  0001 C CNN
 	2    9250 2500
@@
 F 0 "U6" H 9150 2300 50  0000 C CNN
 F 1 "74LS32" H 9450 2300 50  0000 C CNN
-F 2 "" H 9250 2100 50  0001 C CNN
+F 2 "Package_SO:SOIC-14_3.9x8.7mm_P1.27mm" H 9250 2100 50  0001 C CNN
 F 3 "http://www.ti.com/lit/gpn/sn74LS32" H 9250 2100 50  0001 C CNN
 	1    9250 2100
@@
 Wire Wire Line
 	7150 2100 7350 2100
+$Comp
+L Connector:TestPoint_Probe TP1
+U 1 1 5DFE4BF6
+P 7300 1450
+F 0 "TP1" H 7453 1551 50  0000 L CNN
+F 1 "TestPoint_Probe" H 7453 1460 50  0000 L CNN
+F 2 "TestPoint:TestPoint_Pad_D1.5mm" H 7500 1450 50  0001 C CNN
+F 3 "~" H 7500 1450 50  0001 C CNN
+	1    7300 1450
+	1    0    0    -1
+$EndComp
+Wire Wire Line
+	6800 1900 7300 1900
+Wire Wire Line
+	7300 1450 7300 1900
+Connection ~ 7300 1900
+Wire Wire Line
+	7300 1900 7350 1900
 Wire Bus Line
 	4350 5750 4350 6450
 Wire Bus Line
 	4350 4050 4350 5550
+$Comp
+L CPU:Z80CPU U?
+U 1 1 5D5CF86D
+P 3200 5350
+AR Path="/5D5CF86D" Ref="U?"  Part="1"
+AR Path="/5D5CBDC9/5D5CF86D" Ref="U3"  Part="1"
+F 0 "U3" H 2900 6750 50  0000 C CNN
+F 1 "Z80CPU" H 3450 6750 50  0000 C CNN
+F 2 "Package_DIP:DIP-40_W15.24mm" H 3200 5750 50  0001 C CNN
+F 3 "www.zilog.com/manage_directlink.php?filepath=docs/z80/um0080" H 3200 5750 50  0001 C CNN
+	1    3200 5350
+	1    0    0    -1
+$EndComp
 $EndSCHEMATC

Commit message: Schematic updates
Parts:
- removed C5: 0.1u, Capacitor_SMD:C_0603_1608Metric_Pad1.05x0.95mm_HandSolder, symbol Device:C
- removed U3: Z80CPU, Package_DIP:DIP-40_W15.24mm, symbol CPU:Z80CPU
- removed U4: 74LS32, Package_SO:SOIC-14_3.9x8.7mm_P1.27mm, symbol 74xx:74LS32
- removed unit 3 of U6
- added R6: 1k, Resistor_SMD:R_0603_1608Metric_Pad1.05x0.95mm_HandSolder, symbol Device:R
- renumbered R4 to R7, TP1 to TP3, U11 to U10, U6 to U11, U2 to U3, U8 to U5, U9 to U6, U10 to U8, U12 to U9
Connections:
- net +5V: now also R6.2
- net -INT_LD-: no longer names the net of U5.6 (E3)
- net -INT_LD-: now also R6.1
- net ROMDis renamed ROM_DIS
Other:
- moved on the sheet: R7, R8, TP3, U10A, U11A, U11B, U3D, U5, U6A, U6C, U7C, U8D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
