File: schematics/full-schematic/Sheet1.sch (KiCad schematic (older format))
At the start: 32 parts, among them SW1 SW_Push_Dual, SW2 SW_Push_Dual, SW3 SW_SPST, SW4 SW_SPDT, U1 LP3470, U2 74LS04, U3 L7805, U4 Z80CPU, X1 CXO_DIP8

Commit message: Stuff
Parts:
- removed C3, C6: 0.1u, Capacitor_SMD:C_0603_1608Metric_Pad1.05x0.95mm_HandSolder, symbol Device:C
- removed D2: D_Schottky, Diode_SMD:D_0603_1608Metric_Pad1.05x0.95mm_HandSolder, symbol Device:D_Schottky
- removed R4: 10k, Resistor_SMD:R_0603_1608Metric_Pad1.05x0.95mm_HandSolder, symbol Device:R
- removed SW1: SW_Push_Dual, Button_Switch_SMD:SW_MEC_5GSH9, symbol Switch:SW_Push_Dual
- removed SW4: SW_SPDT, Button_Switch_THT:SW_CuK_JS202011CQN_DPDT_Straight, symbol Switch:SW_SPDT
- removed U2: 74LS04, Package_SO:SOIC-14_3.9x8.7mm_P1.27mm, symbol 74xx:74LS04
- removed X1: CXO_DIP8, Oscillator:Oscillator_DIP-8_LargePads, symbol Oscillator:CXO_DIP8
- added C4: 0.1u, Capacitor_SMD:C_0603_1608Metric_Pad1.05x0.95mm_HandSolder, symbol Device:C
- added U2: 74LVC1G08, Package_TO_SOT_SMD:SOT-23-5_HandSoldering, symbol 74xGxx:74LVC1G08
- added X1: XO32, Oscillator:Oscillator_SMD_EuroQuartz_XO32-4Pin_3.2x2.5mm, symbol Oscillator:XO32
- R3: value 100k -> 10k
- SW1: renamed from SW2; footprint Button_Switch_SMD:SW_MEC_5GSH9 -> Button_Switch_THT:SW_PUSH_6mm
- renumbered C4 to C3, C7 to C6, C8 to C7, C9 to C8, D3 to D2, R5 to R4, R17 to R5, R18 to R6, R19 to R7, R20 to R8, SW3 to SW2
Connections:
- net +5V: now also R2.2, U2.5 (VCC), X1.1 (EN), X1.4 (V+); no longer R3.2
- net -RST-: now also U2.4
- net GND: now also C4.2, U2.3 (GND), X1.2 (GND)
- net SYS_CLK: now also X1.3 (OUT)
- net -POR-: now reaches R2.1
- net -POR-: now also U1.5 (-POR-), U2.1
- net at R1.1: now also R3.2, SW1.2, SW1.4; no longer R2.2
- new net: C4.1, R3.1, U2.2
Other:
- moved on the sheet: C1, C2, C3, C5, C6, C7, D1, D2, R4, SW1, SW2, TP2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
