File: schematics/full-schematic/Sheet2.sch (KiCad schematic (older format))
At the start: 18 parts, among them U10 74LS08, U12 74LS04, U13 AT28C256-15PU, U5 74LS138, U6 CY62128ELL-45SXI, U7 74LS32, U8 74LS32, U9 74HC107D

Commit message: Stuff
Parts:
- removed U10: 74LS08, Package_SO:SOIC-14_3.9x8.7mm_P1.27mm, symbol 74xx:74LS08
- removed U12: 74LS04, Package_SO:SOIC-14_3.9x8.7mm_P1.27mm, symbol 74xx:74LS04
- removed U7, U8: 74LS32, Package_SO:SOIC-14_3.9x8.7mm_P1.27mm, symbol 74xx:74LS32
- added U11, U13, U14, U7, U8: 74LVC1G32, Package_TO_SOT_SMD:SOT-23-5_HandSoldering, symbol 74xGxx:74LVC1G32
- added U12: 74LVC1G04, Package_TO_SOT_SMD:SOT-23-5_HandSoldering, symbol 74xGxx:74LVC1G04
- added U9: 74LVC1G08, Package_TO_SOT_SMD:SOT-23-5_HandSoldering, symbol 74xGxx:74LVC1G08
- renumbered C11 to C10, C10 to C9, R7 to R10, R8 to R11, R10 to R12, R9 to R13, R11 to R14, R6 to R9, U9 to U10, U13 to U15
Connections:
- net -IOCS2- is gone; now on net -CFCS-: U5.13 (O2)
- net +5V: now also U11.5 (VCC), U12.5 (VCC), U13.5 (VCC), U14.5 (VCC), U7.5 (VCC), U8.5 (VCC), U9.5 (VCC)
- net -CFCS-: no longer U5.15 (O0)
- net -MREQ-: now also U13.2, U14.1
- net -RAMCS-: now also U14.4
- net -RD-: now also U8.2
- net -ROMCS-: now also U13.4
- net -RST-: now also U9.2
- net -WR-: now also U7.2
- net A15: now also U11.2
- net GND: now also U11.3 (GND), U12.3 (GND), U13.3 (GND), U14.3 (GND), U7.3 (GND), U8.3 (GND), U9.3 (GND)
- net ROM_DIS: now also U11.1
- net at U10.12 (~C): now also U7.4
- net at U10.13 (~R): now also U9.4
- net at U5.7 (O7): now also U7.1, U8.1
- net -IOCS1- renamed -UARTCS-
- new net: U11.4, U12.2, U13.1
- new net: U12.4, U14.2
- new net: U8.4, U9.1
- new net -I2CCS-: U5.15 (O0)
