File: schematics/full-schematic/Sheet3.sch (KiCad schematic (older format))
At the start: 7 parts, among them J1 Conn_02x25_Top_Bottom

Commit message: Stuff
Parts:
- removed R12, R13: 1k, Resistor_SMD:R_0603_1608Metric_Pad1.05x0.95mm_HandSolder, symbol Device:R
- added C11, C12: 0.1u, Capacitor_SMD:C_0603_1608Metric_Pad1.05x0.95mm_HandSolder, symbol Device:C
- added J2, J4: Conn_01x02, Connector_PinHeader_2.54mm:PinHeader_1x02_P2.54mm_Vertical, symbol Connector_Generic:Conn_01x02
- added J3: Conn_01x04, Connector_PinHeader_2.54mm:PinHeader_1x04_P2.54mm_Vertical, symbol Connector_Generic:Conn_01x04
- added R18, R19: 1k, Resistor_SMD:R_0603_1608Metric_Pad1.05x0.95mm_HandSolder, symbol Device:R
- added U16: PCF8584, Package_SO:SOIC-20W_7.5x12.8mm_P1.27mm, symbol z80-project:PCF8584
- added U17: CP82C52Z, Package_DIP:DIP-28_W15.24mm, symbol z80-project:CP82C52Z
- added U18: 74LVC1G04, Package_TO_SOT_SMD:SOT-23-5_HandSoldering, symbol 74xGxx:74LVC1G04
- R15: value 580 -> 1k
- renumbered D4 to D3, R14 to R17
Connections:
- net +5V: now also C11.1, C12.1, R18.1, R19.1, U16.20 (VCC), U17.27 (VCC), U18.5 (VCC)
- net -RD-: now also U16.16 (~RD), U17.1 (~RD)
- net -RST-: now also U16.19 (~RST), U18.2
- net -WR-: now also U16.18 (~WR), U17.2 (~WR)
- net A0: now also U16.6 (A0), U17.11 (A0)
- net A1: now also U17.12 (A1)
- net D0: now also U16.7 (D0), U17.3 (D0)
- net D1: now also U16.8 (D1), U17.4 (D1)
- net D2: now also U16.9 (D2), U17.5 (D2)
- net D3: now also U16.11 (D3), U17.6 (D3)
- net D4: now also U16.12 (D4), U17.7 (D4)
- net D5: now also U16.13 (D5), U17.8 (D5)
- net D6: now also U16.14 (D6), U17.9 (D6)
- net D7: now also U16.15 (D7), U17.10 (D7)
- net GND: now also C11.2, C12.2, U16.10 (GND), U17.16 (GND), U18.3 (GND)
- net at D3.2 (A): now also R18.2; no longer R15.2
- net at J1.46 (Pin_46): now also R19.2; no longer R16.2
- net at J1.36 (Pin_36): now also R16.2
- net at J1.32 (Pin_32): now also R15.2
- new net: J4.2 (Pin_2), U17.15 (Tx)
- new net: J3.4 (Pin_4), U17.17 (~CTS)
- new net: J3.3 (Pin_3), U17.18 (~DSR)
- new net: J3.2 (Pin_2), U17.19 (~DTR)
- new net: J3.1 (Pin_1), U17.20 (~RTS)
- new net: U17.23 (RST), U18.4
- new net: J4.1 (Pin_1), U17.25 (Rx)
- new net -I2CCS-: U16.17 (~CS)
- new net -UARTCS-: U17.28 (~CSO)
- new net SCL: J2.1 (Pin_1), U16.3 (SCL)
- new net SDA: J2.2 (Pin_2), U16.2 (SDA)
- new net SYS_CLK: U16.1 (CLK), U17.13 (IX)
Other:
- moved on the sheet: D3, J1, R17
